Commit message: rename names of robot and joints

File: sample/fullset_robot.urdf (robot description, URDF)
Before this commit: robot AssembleRobot, 47 links, 46 joints
Links:
- link Bottom_mounter_213_18: geometry collision mesh filename=file:///tmp/fullset_robot_Bottom_mounter_213_18_col.stl; visual mesh filename=file:///tmp/fullset_robot_Bottom_mounter_213_18_vis.dae
- link FR12_H103_S_213_23: geometry collision mesh filename=file:///tmp/fullset_robot_FR12_H103_S_213_23_col.stl; visual mesh filename=file:///tmp/fullset_robot_FR12_H103_S_213_23_vis.dae
- link FR12_S102_P_213_1: geometry collision mesh filename=file:///tmp/fullset_robot_FR12_S102_P_213_1_col.stl; visual mesh filename=file:///tmp/fullset_robot_FR12_S102_P_213_1_vis.dae
- link FR12_S102_P_213_2: geometry collision mesh filename=file:///tmp/fullset_robot_FR12_S102_P_213_2_col.stl; visual mesh filename=file:///tmp/fullset_robot_FR12_S102_P_213_2_vis.dae
- link FR12_S102_P_213_25: geometry collision mesh filename=file:///tmp/fullset_robot_FR12_S102_P_213_25_col.stl; visual mesh filename=file:///tmp/fullset_robot_FR12_S102_P_213_25_vis.dae
- link FR12_S102_P_213_3: geometry collision mesh filename=file:///tmp/fullset_robot_FR12_S102_P_213_3_col.stl; visual mesh filename=file:///tmp/fullset_robot_FR12_S102_P_213_3_vis.dae
- link FR12_S102_P_213_4: geometry collision mesh filename=file:///tmp/fullset_robot_FR12_S102_P_213_4_col.stl; visual mesh filename=file:///tmp/fullset_robot_FR12_S102_P_213_4_vis.dae
- link Fixed_Finger_213_26: geometry collision mesh filename=file:///tmp/fullset_robot_Fixed_Finger_213_26_col.stl; visual mesh filename=file:///tmp/fullset_robot_Fixed_Finger_213_26_vis.dae
- link LINK_0: geometry collision mesh filename=file:///tmp/fullset_robot_LINK_0_col.stl; visual mesh filename=file:///tmp/fullset_robot_LINK_0_vis.dae
- link LINK_1: mass 5.695000000000e-03 -> 5.733000000000e-03; geometry collision mesh filename=file:///tmp/fullset_robot_LINK_1_col.stl; visual mesh filename=file:///tmp/fullset_robot_LINK_1_vis.dae
- link LINK_2: mass 1.439500000000e-02 -> 5.695000000000e-03; geometry collision mesh filename=file:///tmp/fullset_robot_LINK_2_col.stl; visual mesh filename=file:///tmp/fullset_robot_LINK_2_vis.dae
- link LINK_3: mass 5.700000000000e-02 -> 1.439500000000e-02; geometry collision mesh filename=file:///tmp/fullset_robot_LINK_3_col.stl; visual mesh filename=file:///tmp/fullset_robot_LINK_3_vis.dae
- link LINK_4: mass 2.395900000000e-02 -> 5.700000000000e-02; geometry collision mesh filename=file:///tmp/fullset_robot_LINK_4_col.stl; visual mesh filename=file:///tmp/fullset_robot_LINK_4_vis.dae
- link LINK_5: mass 5.733000000000e-03 -> 2.395900000000e-02; geometry collision mesh filename=file:///tmp/fullset_robot_LINK_5_col.stl; visual mesh filename=file:///tmp/fullset_robot_LINK_5_vis.dae
- link LINK_6: geometry collision mesh filename=file:///tmp/fullset_robot_LINK_6_col.stl; visual mesh filename=file:///tmp/fullset_robot_LINK_6_vis.dae
- link LINK_7: geometry collision mesh filename=file:///tmp/fullset_robot_LINK_7_col.stl; visual mesh filename=file:///tmp/fullset_robot_LINK_7_vis.dae
- link Root: geometry collision mesh filename=file:///tmp/fullset_robot_Root_col.stl; visual mesh filename=file:///tmp/fullset_robot_Root_vis.dae
- link XL-430_213_19: geometry collision mesh filename=file:///tmp/fullset_robot_XL-430_213_19_col.stl; visual mesh filename=file:///tmp/fullset_robot_XL-430_213_19_vis.dae
- link XL-430_213_21: geometry collision mesh filename=file:///tmp/fullset_robot_XL-430_213_21_col.stl; visual mesh filename=file:///tmp/fullset_robot_XL-430_213_21_vis.dae
- link XL-430_213_27: geometry collision mesh filename=file:///tmp/fullset_robot_XL-430_213_27_col.stl; visual mesh filename=file:///tmp/fullset_robot_XL-430_213_27_vis.dae
- link XL-430_213_5: geometry collision mesh filename=file:///tmp/fullset_robot_XL-430_213_5_col.stl; visual mesh filename=file:///tmp/fullset_robot_XL-430_213_5_vis.dae
- link XL-430_213_6: geometry collision mesh filename=file:///tmp/fullset_robot_XL-430_213_6_col.stl; visual mesh filename=file:///tmp/fullset_robot_XL-430_213_6_vis.dae
- link XL-430_213_7: geometry collision mesh filename=file:///tmp/fullset_robot_XL-430_213_7_col.stl; visual mesh filename=file:///tmp/fullset_robot_XL-430_213_7_vis.dae
- link XL-430_213_8: geometry collision mesh filename=file:///tmp/fullset_robot_XL-430_213_8_col.stl; visual mesh filename=file:///tmp/fullset_robot_XL-430_213_8_vis.dae
- link angle_2_2_5635_0: geometry collision mesh filename=file:///tmp/fullset_robot_angle_2_2_5635_0_col.stl; visual mesh filename=file:///tmp/fullset_robot_angle_2_2_5635_0_vis.dae
- link omni-wheel_213_14: geometry collision mesh filename=file:///tmp/fullset_robot_omni-wheel_213_14_col.stl; visual mesh filename=file:///tmp/fullset_robot_omni-wheel_213_14_vis.dae
- link omni-wheel_213_15: geometry collision mesh filename=file:///tmp/fullset_robot_omni-wheel_213_15_col.stl; visual mesh filename=file:///tmp/fullset_robot_omni-wheel_213_15_vis.dae
- link omni-wheel_213_16: geometry collision mesh filename=file:///tmp/fullset_robot_omni-wheel_213_16_col.stl; visual mesh filename=file:///tmp/fullset_robot_omni-wheel_213_16_vis.dae
- link omni-wheel_213_17: geometry collision mesh filename=file:///tmp/fullset_robot_omni-wheel_213_17_col.stl; visual mesh filename=file:///tmp/fullset_robot_omni-wheel_213_17_vis.dae
- link sensor-mounter_5635_1: geometry collision mesh filename=file:///tmp/fullset_robot_sensor-mounter_5635_1_col.stl; visual mesh filename=file:///tmp/fullset_robot_sensor-mounter_5635_1_vis.dae
- link tof-sensor_5635_2: geometry collision mesh filename=file:///tmp/fullset_robot_tof-sensor_5635_2_col.stl; visual mesh filename=file:///tmp/fullset_robot_tof-sensor_5635_2_vis.dae
- link vehicle-base-ps_213_44: geometry collision mesh filename=file:///tmp/fullset_robot_vehicle-base-ps_213_44_col.stl; visual mesh filename=file:///tmp/fullset_robot_vehicle-base-ps_213_44_vis.dae
Joints:
- removed joint LINK_0
- removed joint LINK_1
- removed joint LINK_2
- removed joint LINK_3
- removed joint LINK_4
- removed joint LINK_5
- removed joint LINK_6
- removed joint LINK_7
- added joint JOINT0: type revolute, parent XL-430_213_19, child LINK_2, origin xyz=1.100000000000e-02 -8.000000000000e-03 -3.600000000000e-02 rpy=3.141592653590e+00 -1.224646799147e-16 3.141592653590e+00, axis 0.000000000000e+00 0.000000000000e+00 1.000000000000e+00, limit lower=-3.141592653590e+00 upper=3.141592653590e+00 effort=1.797693134862e+308 velocity=1.797693134862e+308
- added joint JOINT1: type revolute, parent XL-430_213_21, child LINK_3, origin xyz=3.200000000000e-02 -1.100000000000e-02 2.000000000000e-03 rpy=-1.300702098501e-16 7.850500000000e-17 -1.570796326795e+00, axis 0.000000000000e+00 0.000000000000e+00 1.000000000000e+00, limit lower=-3.141592653590e+00 upper=3.141592653590e+00 effort=1.797693134862e+308 velocity=1.797693134862e+308
- added joint JOINT2: type revolute, parent FR12_H103_S_213_23, child LINK_4, origin xyz=7.000000000000e-03 8.000000000000e-03 5.920000000000e-02 rpy=-1.570796326795e+00 1.110223024625e-16 -1.570796326795e+00, axis -0.000000000000e+00 -0.000000000000e+00 -1.000000000000e+00, limit lower=-3.141592653590e+00 upper=3.141592653590e+00 effort=1.797693134862e+308 velocity=1.797693134862e+308
- added joint JOINT3: type revolute, parent XL-430_213_27, child LINK_5, origin xyz=3.200000000000e-02 -1.100000000000e-02 2.000000000000e-03 rpy=1.684066670566e-16 -3.920331988683e-16 -1.570796326795e+00, axis 0.000000000000e+00 0.000000000000e+00 1.000000000000e+00, limit lower=-3.141592653590e+00 upper=3.141592653590e+00 effort=1.797693134862e+308 velocity=1.797693134862e+308
- added joint WHEEL0: type revolute, parent XL-430_213_6, child LINK_0, origin xyz=3.200000000000e-02 -1.100000000000e-02 2.000000000000e-03 rpy=-3.140180000000e-16 -2.465190328816e-32 1.570796326795e+00, axis 0.000000000000e+00 0.000000000000e+00 1.000000000000e+00, limit lower=-3.141592653590e+00 upper=3.141592653590e+00 effort=1.797693134862e+308 velocity=1.797693134862e+308
- added joint WHEEL1: type revolute, parent XL-430_213_8, child LINK_1, origin xyz=3.200000000000e-02 -1.100000000000e-02 2.000000000000e-03 rpy=3.981020970777e-16 7.850510000000e-17 -1.570796326795e+00, axis 0.000000000000e+00 0.000000000000e+00 1.000000000000e+00, limit lower=-3.141592653590e+00 upper=3.141592653590e+00 effort=1.797693134862e+308 velocity=1.797693134862e+308
- added joint WHEEL2: type revolute, parent XL-430_213_7, child LINK_6, origin xyz=3.200000000000e-02 -1.100000000000e-02 2.000000000000e-03 rpy=-1.648597000000e-15 7.850500000000e-17 -1.570796326795e+00, axis 0.000000000000e+00 0.000000000000e+00 1.000000000000e+00, limit lower=-3.141592653590e+00 upper=3.141592653590e+00 effort=1.797693134862e+308 velocity=1.797693134862e+308
- added joint WHEEL3: type revolute, parent XL-430_213_5, child LINK_7, origin xyz=3.200000000000e-02 -1.100000000000e-02 2.000000000000e-03 rpy=7.121209275474e-16 1.570090000000e-16 -1.570796326795e+00, axis 0.000000000000e+00 0.000000000000e+00 1.000000000000e+00, limit lower=-3.141592653590e+00 upper=3.141592653590e+00 effort=1.797693134862e+308 velocity=1.797693134862e+308
- joint FR12_H103_S_213_23: parent LINK_2 -> LINK_3
- joint FR12_S102_P_213_25: parent LINK_3 -> LINK_4
- joint XL-430_213_21: parent LINK_1 -> LINK_2
- joint omni-wheel_213_14: origin xyz=2.367534269115e-30 -8.491693428602e-19 3.000000000000e-02 rpy=0.000000000000e+00 -3.007574964758e-32 0.000000000000e+00 -> xyz=2.269661440030e-36 2.620277609093e-18 3.000000000000e-02 rpy=0.000000000000e+00 -3.007574964758e-32 0.000000000000e+00; parent LINK_6 -> LINK_0
- joint omni-wheel_213_15: origin xyz=-1.648038893364e-33 9.513175260716e-19 3.000000000000e-02 rpy=-1.554311692010e-15 -8.194292652983e-29 5.047477198250e-29 -> xyz=-2.763898138422e-33 7.890211429979e-18 3.000000000000e-02 rpy=-1.554311692010e-15 -8.194292652983e-29 5.047477198250e-29; parent LINK_5 -> LINK_6
- joint omni-wheel_213_16: origin xyz=6.661470000000e-18 1.971479772646e-17 3.000000000000e-02 rpy=5.551115123126e-16 -5.392603844284e-32 -4.930380657631e-32 -> xyz=2.427408861540e-19 1.971479772646e-17 3.000000000000e-02 rpy=5.551115123126e-16 -5.392603844284e-32 -4.930380657631e-32; parent LINK_7 -> LINK_1
- joint omni-wheel_213_17: origin xyz=5.045021919690e-33 1.872705143085e-17 3.000000000000e-02 rpy=5.551115123126e-16 -1.232595164408e-31 -7.395570986447e-32 -> xyz=4.532141979482e-33 1.525739272065e-17 3.000000000000e-02 rpy=5.551115123126e-16 -1.232595164408e-31 -7.395570986447e-32; parent LINK_0 -> LINK_7

Commit message: add the same name as the joint to the link

File: sample/fullset_robot.urdf (robot description, URDF)
Before this commit: robot fullset_robot, 47 links, 46 joints
Links:
- removed link LINK_0
- removed link LINK_1
- removed link LINK_2
- removed link LINK_3
- removed link LINK_4
- removed link LINK_5
- removed link LINK_6
- removed link LINK_7
- added link JOINT0, mass 5.695000000000e-03; collision mesh filename=file:///tmp/fullset_robot_JOINT0_col.stl; visual mesh filename=file:///tmp/fullset_robot_JOINT0_vis.dae
- added link JOINT1, mass 1.439500000000e-02; collision mesh filename=file:///tmp/fullset_robot_JOINT1_col.stl; visual mesh filename=file:///tmp/fullset_robot_JOINT1_vis.dae
- added link JOINT2, mass 5.700000000000e-02; collision mesh filename=file:///tmp/fullset_robot_JOINT2_col.stl; visual mesh filename=file:///tmp/fullset_robot_JOINT2_vis.dae
- added link JOINT3, mass 2.395900000000e-02; collision mesh filename=file:///tmp/fullset_robot_JOINT3_col.stl; visual mesh filename=file:///tmp/fullset_robot_JOINT3_vis.dae
- added link WHEEL0, mass 5.733000000000e-03; collision mesh filename=file:///tmp/fullset_robot_WHEEL0_col.stl; visual mesh filename=file:///tmp/fullset_robot_WHEEL0_vis.dae
- added link WHEEL1, mass 5.733000000000e-03; collision mesh filename=file:///tmp/fullset_robot_WHEEL1_col.stl; visual mesh filename=file:///tmp/fullset_robot_WHEEL1_vis.dae
- added link WHEEL2, mass 5.733000000000e-03; collision mesh filename=file:///tmp/fullset_robot_WHEEL2_col.stl; visual mesh filename=file:///tmp/fullset_robot_WHEEL2_vis.dae
- added link WHEEL3, mass 5.733000000000e-03; collision mesh filename=file:///tmp/fullset_robot_WHEEL3_col.stl; visual mesh filename=file:///tmp/fullset_robot_WHEEL3_vis.dae
Joints:
- joint FR12_H103_S_213_23: parent LINK_3 -> JOINT1
- joint FR12_S102_P_213_25: parent LINK_4 -> JOINT2
- joint JOINT0: child LINK_2 -> JOINT0
- joint JOINT1: child LINK_3 -> JOINT1
- joint JOINT2: child LINK_4 -> JOINT2
- joint JOINT3: child LINK_5 -> JOINT3
- joint WHEEL0: child LINK_0 -> WHEEL0
- joint WHEEL1: child LINK_1 -> WHEEL1
- joint WHEEL2: child LINK_6 -> WHEEL2
- joint WHEEL3: child LINK_7 -> WHEEL3
- joint XL-430_213_21: parent LINK_2 -> JOINT0
- joint omni-wheel_213_14: parent LINK_0 -> WHEEL0
- joint omni-wheel_213_15: parent LINK_6 -> WHEEL2
- joint omni-wheel_213_16: parent LINK_1 -> WHEEL1
- joint omni-wheel_213_17: parent LINK_7 -> WHEEL3

Commit message: fix joint limits

File: sample/fullset_robot.urdf (robot description, URDF)
Before this commit: robot fullset_robot, 47 links, 46 joints
Joints:
- joint WHEEL0: limit lower=-3.141592653590e+00 upper=3.141592653590e+00 effort=1.797693134862e+308 velocity=1.797693134862e+308 -> lower=-1.797693134862e+308 upper=1.797693134862e+308 effort=1.797693134862e+308 velocity=1.797693134862e+308; type revolute -> continuous
- joint WHEEL1: limit lower=-3.141592653590e+00 upper=3.141592653590e+00 effort=1.797693134862e+308 velocity=1.797693134862e+308 -> lower=-1.797693134862e+308 upper=1.797693134862e+308 effort=1.797693134862e+308 velocity=1.797693134862e+308; type revolute -> continuous
- joint WHEEL2: limit lower=-3.141592653590e+00 upper=3.141592653590e+00 effort=1.797693134862e+308 velocity=1.797693134862e+308 -> lower=-1.797693134862e+308 upper=1.797693134862e+308 effort=1.797693134862e+308 velocity=1.797693134862e+308; type revolute -> continuous
- joint WHEEL3: limit lower=-3.141592653590e+00 upper=3.141592653590e+00 effort=1.797693134862e+308 velocity=1.797693134862e+308 -> lower=-1.797693134862e+308 upper=1.797693134862e+308 effort=1.797693134862e+308 velocity=1.797693134862e+308; type revolute -> continuous

Commit message: add color sensor sample

File: sample/fullset_robot.urdf (robot description, URDF)
Before this commit: robot fullset_robot, 47 links, 46 joints
Links:
- added link block_1_1_3_285_1, mass 2.377730000000e-03; collision box size=8.000000000000e-03 8.000000000000e-03 2.880000000000e-02; visual box size=8.000000000000e-03 8.000000000000e-03 2.880000000000e-02
- added link grove-color-sensor_285_4, mass 2.945000000000e-03; collision mesh filename=file:///tmp/fullset_robot_grove-color-sensor_285_4_col.stl; visual mesh filename=file:///tmp/fullset_robot_grove-color-sensor_285_4_vis.dae
- added link grove-sensor-mounter_285_2, mass 6.297000000000e-03; collision mesh filename=file:///tmp/fullset_robot_grove-sensor-mounter_285_2_col.stl; visual mesh filename=file:///tmp/fullset_robot_grove-sensor-mounter_285_2_vis.dae
- added link plate_2_2_pp_245_0, mass 1.395000000000e-03; collision mesh filename=file:///tmp/fullset_robot_plate_2_2_pp_245_0_col.stl; visual mesh filename=file:///tmp/fullset_robot_plate_2_2_pp_245_0_vis.dae
Joints:
- added joint block_1_1_3_285_1: type fixed, parent plate_2_2_pp_245_0, child block_1_1_3_285_1, origin xyz=0.000000000000e+00 8.000000000000e-03 -3.200000000000e-03 rpy=-3.141592653590e+00 -0.000000000000e+00 0.000000000000e+00
- added joint grove-color-sensor_285_4: type fixed, parent grove-sensor-mounter_285_2, child grove-color-sensor_285_4, origin xyz=0.000000000000e+00 2.094146026542e-18 1.710000000000e-02 rpy=-2.614730000000e-32 -2.465190328816e-32 -1.570796326795e+00
- added joint grove-sensor-mounter_285_2: type fixed, parent block_1_1_3_285_1, child grove-sensor-mounter_285_2, origin xyz=0.000000000000e+00 3.526982781544e-18 2.880000000000e-02 rpy=0.000000000000e+00 -0.000000000000e+00 0.000000000000e+00
- added joint plate_2_2_pp_245_0: type fixed, parent Root, child plate_2_2_pp_245_0, origin xyz=3.200000000000e-02 3.200000000000e-02 0.000000000000e+00 rpy=0.000000000000e+00 -0.000000000000e+00 0.000000000000e+00
- joint WHEEL0: origin xyz=3.200000000000e-02 -1.100000000000e-02 2.000000000000e-03 rpy=-3.140180000000e-16 -2.465190328816e-32 1.570796326795e+00 -> xyz=3.200000000000e-02 -1.100000000000e-02 2.000000000000e-03 rpy=6.280366000000e-16 4.710274000000e-16 1.570796326795e+00
- joint omni-wheel_213_14: origin xyz=2.269661440030e-36 2.620277609093e-18 3.000000000000e-02 rpy=0.000000000000e+00 -3.007574964758e-32 0.000000000000e+00 -> xyz=-2.530341921855e-19 1.006523389737e-17 3.000000000000e-02 rpy=1.776354451335e-15 2.220442225970e-15 1.776354451335e-15
- joint omni-wheel_213_17: origin xyz=4.532141979482e-33 1.525739272065e-17 3.000000000000e-02 rpy=5.551115123126e-16 -1.232595164408e-31 -7.395570986447e-32 -> xyz=7.933930472005e-31 1.525739272065e-17 3.000000000000e-02 rpy=5.551115123126e-16 -1.232595164408e-31 -7.395570986447e-32
